File: Hardware/BRD161205/BRD161205.brd (EAGLE design)
At the start: 73 x 42 mm, 15 parts, among them CN1 MOLEX 4455, U1 TPS73101, U2 PL133-37, U3 74VHC04, X1 10MHz

Commit message: BRD161205 R0
Signed-off-by: Christoph Tack <prog.send@gmail.com>
Parts:
- added DRILEGEND: (no value), drilegend:DRILEGEND
- added R5, R6: 2K4, lieBtrau:RE_1206
- added U$6: (no value), lieBtrau:FR_FRAME_A5
- moved R3 2.55 mm to (11.0, 18.5)
- moved C6 1.50 mm to (14.0, 10.5)
Connections:
- new net N$7: R3.3, R5.1
- new net N$8: R3.1, R6.2
- net 3V0: now also R5.2; no longer R3.1
- net GND: now also R6.1; no longer R3.3
Routing:
- net 3V0: track 29.3 -> 21.1 mm, vias 1 -> 0
- net N$8: track 0.00 -> 6.45 mm, vias 0 -> 1
- net N$7: track 0.00 -> 5.82 mm, vias 0 -> 1
- net GND: track 20.4 -> 24.6 mm
- net N$2: track 11.1 -> 12.5 mm
Other:
- board text added: ">BOARD"
- board text added: ">REV"
